Commit message: rename defs to def

File: def/models.xacro (robot description, xacro)
@@ -2,5 +2,5 @@
 <!--
 Include this to the file you want to use the macros
-	<xacro:include filename="$(find h4r_hardware_models)/defs/models.xacro"/>
+	<xacro:include filename="$(find h4r_hardware_models)/def/models.xacro"/>
 -->
 <robot xmlns:sensor="http://playerstage.sourceforge.net/gazebo/xmlschema/#sensor"
@@ -8,4 +8,4 @@
        xmlns:interface="http://playerstage.sourceforge.net/gazebo/xmlschema/#interface"
        xmlns:xacro="http://ros.org/wiki/xacro">
-       <xacro:include filename="$(find h4r_hardware_models)/defs/sub/delock_96000.xacro"/>
+       <xacro:include filename="$(find h4r_hardware_models)/def/sub/delock_96000.xacro"/>
 </robot>

File: def/sub/delock_96000.xacro (robot description, xacro)
@@ -54,7 +54,5 @@
 has_inertia      ="false"
 >
-<origin xyz="0
-             0
-             -0.0065" rpy="0 ${rr_const_pi/2} ${rr_const_pi/2}" />
+<origin xyz="0 0 -0.0065" rpy="0 ${rr_const_pi/2} ${rr_const_pi/2}" />
 <geometry>
 	<sphere radius="0.0015" />
